File: pcb/Replica_NEO_6M_GPS/Replica_NEO_6M_GPS.kicad_pcb (KiCad board)
At the start: 2 copper layers, 46 x 36 mm, 24 parts, among them J1 CONUFL001-SMD-T, J2 Conn_01x04, U1 TPS79133DBVR, U2 NEO-6M-GPS, U3 24AA32A-I_MS

Commit message: Se hicieron cambiaron los footprints de los LEDS D1,D2
Parts:
- D1, D2: footprint LED_SMD:LED_0201_0603Metric_Pad0.64x0.40mm_HandSolder -> LED_SMD:LED_0805_2012Metric_Pad1.15x1.40mm_HandSolder
- moved D1 0.50 mm to (158.5, 116.5)
- moved D2 0.50 mm to (164.5, 111.5)
Changed lines of the file:
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@@
-    )
-  )
-  (module LED_SMD:LED_0201_0603Metric_Pad0.64x0.40mm_HandSolder (layer F.Cu)
-    (at 158 116.5 180)
-    (descr "LED SMD 0201 (0603 Metric), square (rectangular) end terminal, IPC_7351 nominal, (Body size source: https://www.vishay.com/docs/20052/crcw0201e3.pdf), generated with kicad-footprint-generator")
-    (tags "LED handsolder")
-    (attr smd)
-    (fp_text reference D1 (at 0 -1.05) (layer F.SilkS)
-      (effects (font (size 1 1) (thickness 0.15)))
-    )
-    (fp_text value LED (at 0 1.05) (layer F.Fab)
-      (effects (font (size 1 1) (thickness 0.15)))
-    )
-    (fp_line (start 0.88 0.35) (end -0.88 0.35) (layer F.CrtYd) (width 0.05))
-    (fp_line (start 0.88 -0.35) (end 0.88 0.35) (layer F.CrtYd) (width 0.05))
-    (fp_line (start -0.88 -0.35) (end 0.88 -0.35) (layer F.CrtYd) (width 0.05))
-    (fp_line (start -0.88 0.35) (end -0.88 -0.35) (layer F.CrtYd) (width 0.05))
-    (fp_line (start -0.1 0.15) (end -0.1 -0.15) (layer F.Fab) (width 0.1))
-    (fp_line (start -0.2 0.15) (end -0.2 -0.15) (layer F.Fab) (width 0.1))
-    (fp_line (start 0.3 0.15) (end -0.3 0.15) (layer F.Fab) (width 0.1))
-    (fp_line (start 0.3 -0.15) (end 0.3 0.15) (layer F.Fab) (width 0.1))
-    (fp_line (start -0.3 -0.15) (end 0.3 -0.15) (layer F.Fab) (width 0.1))
-    (fp_line (start -0.3 0.15) (end -0.3 -0.15) (layer F.Fab) (width 0.1))
-    (fp_circle (center -1.035 0) (end -0.985 0) (layer F.SilkS) (width 0.1))
-    (fp_text user %R (at 0 -0.68) (layer F.Fab)
-      (effects (font (size 0.25 0.25) (thickness 0.04)))
-    )
-    (pad "" smd roundrect (at -0.4325 0 180) (size 0.458 0.36) (layers F.Paste) (roundrect_rratio 0.25))
-    (pad "" smd roundrect (at 0.4325 0 180) (size 0.458 0.36) (layers F.Paste) (roundrect_rratio 0.25))
-    (pad 1 smd roundrect (at -0.4075 0 180) (size 0.635 0.4) (layers F.Cu F.Mask) (roundrect_rratio 0.25)
-      (net 2 Earth))
-    (pad 2 smd roundrect (at 0.4075 0 180) (size 0.635 0.4) (layers F.Cu F.Mask) (roundrect_rratio 0.25)
-      (net 6 "Net-(D1-Pad2)"))
-    (model ${KISYS3DMOD}/LED_SMD.3dshapes/LED_0201_0603Metric.wrl
-      (at (xyz 0 0 0))
-      (scale (xyz 1 1 1))
-      (rotate (xyz 0 0 0))
-    )
-  )
-  (module LED_SMD:LED_0201_0603Metric_Pad0.64x0.40mm_HandSolder (layer F.Cu)
-    (at 164.5 111)
-    (descr "LED SMD 0201 (0603 Metric), square (rectangular) end terminal, IPC_7351 nominal, (Body size source: https://www.vishay.com/docs/20052/crcw0201e3.pdf), generated with kicad-footprint-generator")
-    (tags "LED handsolder")
-    (attr smd)
-    (fp_text reference D2 (at 0 -1.05) (layer F.SilkS)
-      (effects (font (size 1 1) (thickness 0.15)))
-    )
-    (fp_text value FIX (at 0 1.05) (layer F.Fab)
-      (effects (font (size 1 1) (thickness 0.15)))
-    )
-    (fp_text user %R (at 0 -0.68) (layer F.Fab)
-      (effects (font (size 0.25 0.25) (thickness 0.04)))
-    )
-    (fp_circle (center -1.035 0) (end -0.985 0) (layer F.SilkS) (width 0.1))
-    (fp_line (start -0.3 0.15) (end -0.3 -0.15) (layer F.Fab) (width 0.1))
-    (fp_line (start -0.3 -0.15) (end 0.3 -0.15) (layer F.Fab) (width 0.1))
-    (fp_line (start 0.3 -0.15) (end 0.3 0.15) (layer F.Fab) (width 0.1))
-    (fp_line (start 0.3 0.15) (end -0.3 0.15) (layer F.Fab) (width 0.1))
-    (fp_line (start -0.2 0.15) (end -0.2 -0.15) (layer F.Fab) (width 0.1))
-    (fp_line (start -0.1 0.15) (end -0.1 -0.15) (layer F.Fab) (width 0.1))
-    (fp_line (start -0.88 0.35) (end -0.88 -0.35) (layer F.CrtYd) (width 0.05))
-    (fp_line (start -0.88 -0.35) (end 0.88 -0.35) (layer F.CrtYd) (width 0.05))
-    (fp_line (start 0.88 -0.35) (end 0.88 0.35) (layer F.CrtYd) (width 0.05))
-    (fp_line (start 0.88 0.35) (end -0.88 0.35) (layer F.CrtYd) (width 0.05))
-    (pad 2 smd roundrect (at 0.4075 0) (size 0.635 0.4) (layers F.Cu F.Mask) (roundrect_rratio 0.25)
-      (net 7 "Net-(D2-Pad2)"))
-    (pad 1 smd roundrect (at -0.4075 0) (size 0.635 0.4) (layers F.Cu F.Mask) (roundrect_rratio 0.25)
-      (net 2 Earth))
-    (pad "" smd roundrect (at 0.4325 0) (size 0.458 0.36) (layers F.Paste) (roundrect_rratio 0.25))
-    (pad "" smd roundrect (at -0.4325 0) (size 0.458 0.36) (layers F.Paste) (roundrect_rratio 0.25))
-    (model ${KISYS3DMOD}/LED_SMD.3dshapes/LED_0201_0603Metric.wrl
-      (at (xyz 0 0 0))
-      (scale (xyz 1 1 1))
-      (rotate (xyz 0 0 0))
     )
   )
@@
     (pad 1 np_thru_hole circle (at 0 0) (size 4 4) (drill 4) (layers *.Cu *.Mask))
   )
+  (module LED_SMD:LED_0805_2012Metric_Pad1.15x1.40mm_HandSolder (layer F.Cu)
+    (at 158.5 116.5 180)
+    (descr "LED SMD 0805 (2012 Metric), square (rectangular) end terminal, IPC_7351 nominal, (Body size source: https://docs.google.com/spreadsheets/d/1BsfQQcO9C6DZCsRaXUlFlo91Tg2WpOkGARC1WS5S8t0/edit?usp=sharing), generated with kicad-footprint-generator")
+    (tags "LED handsolder")
+    (attr smd)
+    (fp_text reference D1 (at 0 -1.65) (layer F.SilkS)
+      (effects (font (size 1 1) (thickness 0.15)))
+    )
+    (fp_text value LED (at 0 1.65) (layer F.Fab)
+      (effects (font (size 1 1) (thickness 0.15)))
+    )
+    (fp_line (start 1.85 0.95) (end -1.85 0.95) (layer F.CrtYd) (width 0.05))
+    (fp_line (start 1.85 -0.95) (end 1.85 0.95) (layer F.CrtYd) (width 0.05))
+    (fp_line (start -1.85 -0.95) (end 1.85 -0.95) (layer F.CrtYd) (width 0.05))
+    (fp_line (start -1.85 0.95) (end -1.85 -0.95) (layer F.CrtYd) (width 0.05))
+    (fp_line (start -1.86 0.96) (end 1 0.96) (layer F.SilkS) (width 0.12))
+    (fp_line (start -1.86 -0.96) (end -1.86 0.96) (layer F.SilkS) (width 0.12))
+    (fp_line (start 1 -0.96) (end -1.86 -0.96) (layer F.SilkS) (width 0.12))
+    (fp_line (start 1 0.6) (end 1 -0.6) (layer F.Fab) (width 0.1))
+    (fp_line (start -1 0.6) (end 1 0.6) (layer F.Fab) (width 0.1))
+    (fp_line (start -1 -0.3) (end -1 0.6) (layer F.Fab) (width 0.1))
+    (fp_line (start -0.7 -0.6) (end -1 -0.3) (layer F.Fab) (width 0.1))
+    (fp_line (start 1 -0.6) (end -0.7 -0.6) (layer F.Fab) (width 0.1))
+    (fp_text user %R (at 0 0) (layer F.Fab)
+      (effects (font (size 0.5 0.5) (thickness 0.08)))
+    )
+    (pad 1 smd roundrect (at -1.025 0 180) (size 1.15 1.4) (layers F.Cu F.Paste F.Mask) (roundrect_rratio 0.217391)
+      (net 2 Earth))
+    (pad 2 smd roundrect (at 1.025 0 180) (size 1.15 1.4) (layers F.Cu F.Paste F.Mask) (roundrect_rratio 0.217391)
+      (net 6 "Net-(D1-Pad2)"))
+    (model ${KISYS3DMOD}/LED_SMD.3dshapes/LED_0805_2012Metric.wrl
+      (at (xyz 0 0 0))
+      (scale (xyz 1 1 1))
+      (rotate (xyz 0 0 0))
+    )
+  )
+  (module LED_SMD:LED_0805_2012Metric_Pad1.15x1.40mm_HandSolder (layer F.Cu)
+    (at 164.5 111.5)
+    (descr "LED SMD 0805 (2012 Metric), square (rectangular) end terminal, IPC_7351 nominal, (Body size source: https://docs.google.com/spreadsheets/d/1BsfQQcO9C6DZCsRaXUlFlo91Tg2WpOkGARC1WS5S8t0/edit?usp=sharing), generated with kicad-footprint-generator")
+    (tags "LED handsolder")
+    (attr smd)
+    (fp_text reference D2 (at 0 -1.65) (layer F.SilkS)
+      (effects (font (size 1 1) (thickness 0.15)))
+    )
+    (fp_text value FIX (at 0 1.65) (layer F.Fab)
+      (effects (font (size 1 1) (thickness 0.15)))
+    )
+    (fp_text user %R (at 0 0) (layer F.Fab)
+      (effects (font (size 0.5 0.5) (thickness 0.08)))
+    )
+    (fp_line (start 1 -0.6) (end -0.7 -0.6) (layer F.Fab) (width 0.1))
+    (fp_line (start -0.7 -0.6) (end -1 -0.3) (layer F.Fab) (width 0.1))
+    (fp_line (start -1 -0.3) (end -1 0.6) (layer F.Fab) (width 0.1))
+    (fp_line (start -1 0.6) (end 1 0.6) (layer F.Fab) (width 0.1))
+    (fp_line (start 1 0.6) (end 1 -0.6) (layer F.Fab) (width 0.1))
+    (fp_line (start 1 -0.96) (end -1.86 -0.96) (layer F.SilkS) (width 0.12))
+    (fp_line (start -1.86 -0.96) (end -1.86 0.96) (layer F.SilkS) (width 0.12))
+    (fp_line (start -1.86 0.96) (end 1 0.96) (layer F.SilkS) (width 0.12))
+    (fp_line (start -1.85 0.95) (end -1.85 -0.95) (layer F.CrtYd) (width 0.05))
+    (fp_line (start -1.85 -0.95) (end 1.85 -0.95) (layer F.CrtYd) (width 0.05))
+    (fp_line (start 1.85 -0.95) (end 1.85 0.95) (layer F.CrtYd) (width 0.05))
+    (fp_line (start 1.85 0.95) (end -1.85 0.95) (layer F.CrtYd) (width 0.05))
+    (pad 2 smd roundrect (at 1.025 0) (size 1.15 1.4) (layers F.Cu F.Paste F.Mask) (roundrect_rratio 0.217391)
+      (net 7 "Net-(D2-Pad2)"))
+    (pad 1 smd roundrect (at -1.025 0) (size 1.15 1.4) (layers F.Cu F.Paste F.Mask) (roundrect_rratio 0.217391)
+      (net 2 Earth))
+    (model ${KISYS3DMOD}/LED_SMD.3dshapes/LED_0805_2012Metric.wrl
+      (at (xyz 0 0 0))
+      (scale (xyz 1 1 1))
+      (rotate (xyz 0 0 0))
+    )
+  )
   (gr_text "- Se incrementaron las dimensiones del PCB respecto al patron dado que se usan footprints mas grandes\n- NOTAS DE CUADRICULA: Borde del PCB (1mm), Margen del PCB (1mm)\n\n" (at 115.5 127.5) (layer Dwgs.User)
