File: pcb/Replica_NEO_6M_GPS/Replica_NEO_6M_GPS.kicad_pcb (KiCad board)
At the start: 2 copper layers, 36 x 26 mm, 22 parts, among them J1 CONUFL001-SMD-T, J2 Conn_01x04, U1 TPS79133DBVR, U2 24AA32A-I_MS, U3 NEO-6M-GPS

Commit message: Se hiceron correcciones 23/08/2021
Parts:
- removed H5: MountingHole, MountingHole:MountingHole_4mm
- added FID1: Fiducial, Fiducial:Fiducial_0.5mm_Mask1mm, F.Cu at (148.5, 104.5)
- added FID2: Fiducial, Fiducial:Fiducial_0.5mm_Mask1mm, F.Cu at (119.8, 86.5)
- added H6: MountingHole, MountingHole:MountingHole_3.5mm_Pad, F.Cu at (123.0, 93.0)
- added H7: MountingHole, MountingHole:MountingHole_3.5mm_Pad, F.Cu at (141.0, 93.0)
- added H8: MountingHole, MountingHole:MountingHole_3.5mm_Pad, F.Cu at (141.0, 104.0)
- added H9: MountingHole, MountingHole:MountingHole_3.5mm_Pad, F.Cu at (123.0, 104.0)
- C4: value TAJP156M006SNJ -> 4,7uF
- moved C2 3.43 mm to (119.4, 101.5), turned to 270 degrees
- moved R3 3.36 mm to (124.0, 101.5), turned to 90 degrees
- moved B1 0.56 mm to (123.2, 107.2)
- moved C1 0.40 mm to (121.7, 91.4)
- moved C4 0.25 mm to (130.0, 108.5)
- turned D2 to 90 degrees
Routing:
- net Net-(B1-Pad+): track 13.2 -> 24.5 mm
- net GND: track 19.0 -> 21.9 mm, vias 2 -> 0
- net /RXD1: track 27.7 -> 26.4 mm
- net /TXD1: track 24.8 -> 23.9 mm
- net +3V3: track 28.0 -> 28.1 mm, vias 2 -> 0
Other:
- net class Default: trace_width 0.25 -> 0.3; via_dia 0.4 -> 0.8; via_drill 0.3 -> 0.4
- board text added: "3CEIoT UBA Christian Canaan UBA"
- board text added: "Comentarios: - No encuentro el footprint apropiado para la bateria, los que encuentro son mas grandes y no entran en el pcb (ademas de que no se corresponden con la pila que debe ir alli) - Se logro eliminar la necesidad del uso de puentes. Notas: - Componentes 0805 SMD. - Solo se coloco el conector de bateria TH. Bordes y margenes: - Borde de PCB (1 mm) - Margen del PCB (0,5 mm) Cuadriculas de t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"
- board text added: "Réplica uBLOX NEO-6M V2 GPS"
- board text removed: "Comentarios: - No encuentro el footprint apropiado para la bateria, los que encuentro son mas grandes y no entran en el pcb (ademas de que no se corresponden con la pila que debe ir alli) - Fue muy complicado el ruteo sobre U1, el unico modelo que encontre esta espejado respecto a la replica y eso me obligo a usar la otra capa y armar puentes. Bordes y margenes: - Borde de PCB (1 mm) - Margen del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"
- board text removed: "GPS6MV2"
