File: pcb/Replica_NEO_6M_GPS/Replica_NEO_6M_GPS.sch (KiCad schematic (older format))
At the start: 1 part, among them J2 Conn_01x04

Commit message: Se hicieron correcciones y se avanzo con el PCB
Parts:
- added H1, H2, H3, H4: MountingHole, MountingHole:MountingHole_3mm, symbol Mechanical:MountingHole
- added H5: MountingHole, MountingHole:MountingHole_4mm, symbol Mechanical:MountingHole
Other:
- note added: "Hollos para montaje mecanico\n4x3mm\n1x4mm"
Changed lines of the file:
@@
 Text Notes 4550 4300 0    50   ~ 10
 TXD1
+$Comp
+L Mechanical:MountingHole H1
+U 1 1 61193E6F
+P 8400 2250
+F 0 "H1" H 8500 2296 50  0000 L CNN
+F 1 "MountingHole" H 8500 2205 50  0000 L CNN
+F 2 "MountingHole:MountingHole_3mm" H 8400 2250 50  0001 C CNN
+F 3 "~" H 8400 2250 50  0001 C CNN
+	1    8400 2250
+	1    0    0    -1
+$EndComp
+$Comp
+L Mechanical:MountingHole H2
+U 1 1 611942D8
+P 8400 2450
+F 0 "H2" H 8500 2496 50  0000 L CNN
+F 1 "MountingHole" H 8500 2405 50  0000 L CNN
+F 2 "MountingHole:MountingHole_3mm" H 8400 2450 50  0001 C CNN
+F 3 "~" H 8400 2450 50  0001 C CNN
+	1    8400 2450
+	1    0    0    -1
+$EndComp
+$Comp
+L Mechanical:MountingHole H3
+U 1 1 6119459C
+P 8400 2650
+F 0 "H3" H 8500 2696 50  0000 L CNN
+F 1 "MountingHole" H 8500 2605 50  0000 L CNN
+F 2 "MountingHole:MountingHole_3mm" H 8400 2650 50  0001 C CNN
+F 3 "~" H 8400 2650 50  0001 C CNN
+	1    8400 2650
+	1    0    0    -1
+$EndComp
+$Comp
+L Mechanical:MountingHole H4
+U 1 1 611948E2
+P 8400 2850
+F 0 "H4" H 8500 2896 50  0000 L CNN
+F 1 "MountingHole" H 8500 2805 50  0000 L CNN
+F 2 "MountingHole:MountingHole_3mm" H 8400 2850 50  0001 C CNN
+F 3 "~" H 8400 2850 50  0001 C CNN
+	1    8400 2850
+	1    0    0    -1
+$EndComp
+$Comp
+L Mechanical:MountingHole H5
+U 1 1 611961F1
+P 8400 3050
+F 0 "H5" H 8500 3096 50  0000 L CNN
+F 1 "MountingHole" H 8500 3005 50  0000 L CNN
+F 2 "MountingHole:MountingHole_4mm" H 8400 3050 50  0001 C CNN
+F 3 "~" H 8400 3050 50  0001 C CNN
+	1    8400 3050
+	1    0    0    -1
+$EndComp
+Wire Notes Line
+	8250 2050 9100 2050
+Wire Notes Line
+	9100 3250 8250 3250
+Wire Notes Line
+	8250 3250 8250 2050
+Wire Notes Line
+	9100 2050 9100 3250
+Text Notes 9150 2750 0    50   ~ 0
+Hollos para montaje mecanico\n4x3mm\n1x4mm
 $EndSCHEMATC

Commit message: se retoco el esquematico
Connections:
- wire segments 21 -> 20
Other:
- moved on the sheet: H1, H2, H3, H4, H5, J2
Changed lines of the file:
@@
 $EndDescr
 $Sheet
-S 5650 2450 1100 900
+S 2750 2800 1100 900
 U 60EC53CA
 F0 "Regulador de voltaje lineal de potencia" 50
 F1 "Alimentacion.sch" 50
-F2 "3.3V" I R 6750 2900 50
-F3 "+5V" I L 5650 2900 50
-F4 "GND" I R 6750 3250 50
+F2 "3.3V" I R 3850 3250 50
+F3 "+5V" I L 2750 3250 50
+F4 "GND" I R 3850 3600 50
 $EndSheet
 $Sheet
-S 5450 3650 1650 1550
+S 4300 3350 1650 1550
 U 60EC55A9
 F0 "Modulo GPS" 50
 F1 "NEO-6M.sch" 50
-F2 "3.3V" I L 5450 3800 50
-F3 "GND" I R 7100 5050 50
-F4 "TXD1" I L 5450 4300 50
-F5 "RXD1" I L 5450 4200 50
-F6 "SDA2" B R 7100 4450 50
-F7 "SCL2" B R 7100 4600 50
+F2 "3.3V" I L 4300 3500 50
+F3 "GND" I R 5950 4750 50
+F4 "TXD1" I L 4300 4000 50
+F5 "RXD1" I L 4300 3900 50
+F6 "SDA2" B R 5950 4150 50
+F7 "SCL2" B R 5950 4300 50
 $EndSheet
 $Sheet
-S 7550 4050 1050 850
+S 6400 3750 1050 850
 U 60EC55E9
 F0 "Serial EEPROM" 50
 F1 "Memoria.sch" 50
-F2 "GND" I L 7550 4750 50
-F3 "SCL2" B L 7550 4600 50
-F4 "SDA2" B L 7550 4450 50
-F5 "3.3V" I L 7550 4150 50
+F2 "GND" I L 6400 4450 50
+F3 "SCL2" B L 6400 4300 50
+F4 "SDA2" B L 6400 4150 50
+F5 "3.3V" I L 6400 3850 50
 $EndSheet
 $Comp
 L Connector_Generic:Conn_01x04 J?
 U 1 1 60FCF122
-P 4350 4100
+P 1700 3800
 AR Path="/60EC55A9/60FCF122" Ref="J?"  Part="1"
 AR Path="/60FCF122" Ref="J2"  Part="1"
-F 0 "J2" V 4222 3812 50  0000 R CNN
-F 1 "Conn_01x04" V 4313 3812 50  0000 R CNN
-F 2 "Connector_PinHeader_2.54mm:PinHeader_1x04_P2.54mm_Horizontal" H 4350 4100 50  0001 C CNN
-F 3 "~" H 4350 4100 50  0001 C CNN
-	1    4350 4100
+F 0 "J2" V 1572 3512 50  0000 R CNN
+F 1 "Conn_01x04" V 1663 3512 50  0000 R CNN
+F 2 "Connector_PinHeader_2.54mm:PinHeader_1x04_P2.54mm_Horizontal" H 1700 3800 50  0001 C CNN
+F 3 "~" H 1700 3800 50  0001 C CNN
+	1    1700 3800
 	-1   0    0    -1
 $EndComp
 Wire Wire Line
-	4550 4100 5200 4100
+	1900 3800 2550 3800
 Wire Wire Line
-	5200 4100 5200 2900
-Wire Wire Line
-	5200 2900 5650 2900
-Wire Wire Line
-	4550 4000 4850 4000
+	1900 3700 2200 3700
 $Comp
 L power:Earth #PWR0101
 U 1 1 60FD5B75
-P 4850 4000
-F 0 "#PWR0101" H 4850 3750 50  0001 C CNN
-F 1 "Earth" H 4850 3850 50  0001 C CNN
-F 2 "" H 4850 4000 50  0001 C CNN
-F 3 "~" H 4850 4000 50  0001 C CNN
-	1    4850 4000
+P 2200 3700
+F 0 "#PWR0101" H 2200 3450 50  0001 C CNN
+F 1 "Earth" H 2200 3550 50  0001 C CNN
+F 2 "" H 2200 3700 50  0001 C CNN
+F 3 "~" H 2200 3700 50  0001 C CNN
+	1    2200 3700
 	0    -1   -1   0
 $EndComp
@@
 L power:Earth #PWR0102
 U 1 1 60FD674D
-P 7350 5550
-F 0 "#PWR0102" H 7350 5300 50  0001 C CNN
-F 1 "Earth" H 7350 5400 50  0001 C CNN
-F 2 "" H 7350 5550 50  0001 C CNN
-F 3 "~" H 7350 5550 50  0001 C CNN
-	1    7350 5550
+P 6200 5250
+F 0 "#PWR0102" H 6200 5000 50  0001 C CNN
+F 1 "Earth" H 6200 5100 50  0001 C CNN
+F 2 "" H 6200 5250 50  0001 C CNN
+F 3 "~" H 6200 5250 50  0001 C CNN
+	1    6200 5250
 	1    0    0    -1
 $EndComp
@@
 L power:Earth #PWR0103
 U 1 1 60FD7272
-P 7050 3350
-F 0 "#PWR0103" H 7050 3100 50  0001 C CNN
-F 1 "Earth" H 7050 3200 50  0001 C CNN
-F 2 "" H 7050 3350 50  0001 C CNN
-F 3 "~" H 7050 3350 50  0001 C CNN
-	1    7050 3350
+P 4000 3700
+F 0 "#PWR0103" H 4000 3450 50  0001 C CNN
+F 1 "Earth" H 4000 3550 50  0001 C CNN
+F 2 "" H 4000 3700 50  0001 C CNN
+F 3 "~" H 4000 3700 50  0001 C CNN
+	1    4000 3700
 	1    0    0    -1
 $EndComp
 Wire Wire Line
-	6750 3250 7050 3250
+	4000 3600 4000 3700
 Wire Wire Line
-	7050 3250 7050 3350
+	6200 4750 6200 5250
 Wire Wire Line
-	7350 5050 7350 5550
+	5950 4750 6200 4750
 Wire Wire Line
-	7100 5050 7350 5050
+	6400 4450 6200 4450
 Wire Wire Line
-	7550 4750 7350 4750
+	6200 4450 6200 4750
+Connection ~ 6200 4750
 Wire Wire Line
-	7350 4750 7350 5050
-Connection ~ 7350 5050
+	5950 4150 6400 4150
 Wire Wire Line
-	4550 4200 5450 4200
+	5950 4300 6400 4300
 Wire Wire Line
-	4550 4300 5450 4300
+	6200 3850 6400 3850
 Wire Wire Line
-	7100 4450 7550 4450
+	4300 3500 4200 3500
 Wire Wire Line
-	7100 4600 7550 4600
+	4200 3500 4200 3250
 Wire Wire Line
-	6750 2900 7350 2900
+	4200 3250 6200 3250
 Wire Wire Line
-	7350 2900 7350 3550
-Wire Wire Line
-	7350 4150 7550 4150
-Wire Wire Line
-	5450 3800 5350 3800
-Wire Wire Line
-	5350 3800 5350 3550
-Wire Wire Line
-	5350 3550 7350 3550
-Connection ~ 7350 3550
-Wire Wire Line
-	7350 3550 7350 4150
-Text Notes 4550 4000 0    50   ~ 10
+	6200 3250 6200 3850
+Text Notes 1900 3700 0    50   ~ 10
 GND
-Text Notes 4550 4100 0    50   ~ 10
+Text Notes 1900 3800 0    50   ~ 10
 5V
-Text Notes 4550 4200 0    50   ~ 10
+Text Notes 1900 3900 0    50   ~ 10
 RXD1\n
-Text Notes 4550 4300 0    50   ~ 10
+Text Notes 1900 4000 0    50   ~ 10
 TXD1
 $Comp
 L Mechanical:MountingHole H1
 U 1 1 61193E6F
-P 8400 2250
-F 0 "H1" H 8500 2296 50  0000 L CNN
-F 1 "MountingHole" H 8500 2205 50  0000 L CNN
-F 2 "MountingHole:MountingHole_3mm" H 8400 2250 50  0001 C CNN
-F 3 "~" H 8400 2250 50  0001 C CNN
-	1    8400 2250
+P 8200 3850
+F 0 "H1" H 8300 3896 50  0000 L CNN
+F 1 "MountingHole" H 8300 3805 50  0000 L CNN
+F 2 "MountingHole:MountingHole_3mm" H 8200 3850 50  0001 C CNN
+F 3 "~" H 8200 3850 50  0001 C CNN
+	1    8200 3850
 	1    0    0    -1
 $EndComp
@@
 L Mechanical:MountingHole H2
 U 1 1 611942D8
-P 8400 2450
-F 0 "H2" H 8500 2496 50  0000 L CNN
-F 1 "MountingHole" H 8500 2405 50  0000 L CNN
-F 2 "MountingHole:MountingHole_3mm" H 8400 2450 50  0001 C CNN
-F 3 "~" H 8400 2450 50  0001 C CNN
-	1    8400 2450
+P 8200 4050
+F 0 "H2" H 8300 4096 50  0000 L CNN
+F 1 "MountingHole" H 8300 4005 50  0000 L CNN
+F 2 "MountingHole:MountingHole_3mm" H 8200 4050 50  0001 C CNN
+F 3 "~" H 8200 4050 50  0001 C CNN
+	1    8200 4050
 	1    0    0    -1
 $EndComp
@@
 L Mechanical:MountingHole H3
 U 1 1 6119459C
-P 8400 2650
-F 0 "H3" H 8500 2696 50  0000 L CNN
-F 1 "MountingHole" H 8500 2605 50  0000 L CNN
-F 2 "MountingHole:MountingHole_3mm" H 8400 2650 50  0001 C CNN
-F 3 "~" H 8400 2650 50  0001 C CNN
-	1    8400 2650
+P 8200 4250
+F 0 "H3" H 8300 4296 50  0000 L CNN
+F 1 "MountingHole" H 8300 4205 50  0000 L CNN
+F 2 "MountingHole:MountingHole_3mm" H 8200 4250 50  0001 C CNN
+F 3 "~" H 8200 4250 50  0001 C CNN
+	1    8200 4250
 	1    0    0    -1
 $EndComp
@@
 L Mechanical:MountingHole H4
 U 1 1 611948E2
-P 8400 2850
-F 0 "H4" H 8500 2896 50  0000 L CNN
-F 1 "MountingHole" H 8500 2805 50  0000 L CNN
-F 2 "MountingHole:MountingHole_3mm" H 8400 2850 50  0001 C CNN
-F 3 "~" H 8400 2850 50  0001 C CNN
-	1    8400 2850
+P 8200 4450
+F 0 "H4" H 8300 4496 50  0000 L CNN
+F 1 "MountingHole" H 8300 4405 50  0000 L CNN
+F 2 "MountingHole:MountingHole_3mm" H 8200 4450 50  0001 C CNN
+F 3 "~" H 8200 4450 50  0001 C CNN
+	1    8200 4450
 	1    0    0    -1
 $EndComp
@@
 L Mechanical:MountingHole H5
 U 1 1 611961F1
-P 8400 3050
-F 0 "H5" H 8500 3096 50  0000 L CNN
-F 1 "MountingHole" H 8500 3005 50  0000 L CNN
-F 2 "MountingHole:MountingHole_4mm" H 8400 3050 50  0001 C CNN
-F 3 "~" H 8400 3050 50  0001 C CNN
-	1    8400 3050
+P 8200 4650
+F 0 "H5" H 8300 4696 50  0000 L CNN
+F 1 "MountingHole" H 8300 4605 50  0000 L CNN
+F 2 "MountingHole:MountingHole_4mm" H 8200 4650 50  0001 C CNN
+F 3 "~" H 8200 4650 50  0001 C CNN
+	1    8200 4650
 	1    0    0    -1
 $EndComp
 Wire Notes Line
-	8250 2050 9100 2050
+	8050 3650 8900 3650
 Wire Notes Line
-	9100 3250 8250 3250
+	8900 4850 8050 4850
 Wire Notes Line
-	8250 3250 8250 2050
+	8050 4850 8050 3650
 Wire Notes Line
-	9100 2050 9100 3250
-Text Notes 9150 2750 0    50   ~ 0
+	8900 3650 8900 4850
+Text Notes 9000 4300 0    50   ~ 0
 Hollos para montaje mecanico\n4x3mm\n1x4mm
+Wire Wire Line
+	2550 3800 2550 3250
+Wire Wire Line
+	2550 3250 2750 3250
+Wire Wire Line
+	3850 3250 4200 3250
+Connection ~ 4200 3250
+Wire Wire Line
+	1900 3900 4300 3900
+Wire Wire Line
+	1900 4000 4300 4000
+Wire Wire Line
+	3850 3600 4000 3600
 $EndSCHEMATC

Commit message: Se hicieron correcciones
Parts:
- added B1: MS621FE, foot:MS621FE, symbol MS621FE:MS621FE
- added C1, C5: 0.1uF, Capacitor_SMD:C_0805_2012Metric_Pad1.18x1.45mm_HandSolder, symbol Device:C
- added C2: 0.01uF, Capacitor_SMD:C_0805_2012Metric_Pad1.18x1.45mm_HandSolder, symbol Device:C
- added C3: 4.7uF, Capacitor_SMD:C_0805_2012Metric_Pad1.18x1.45mm_HandSolder, symbol Device:C
- added C4: 4.7uF, foot:CAPC2012X140N, symbol TAJP156M006SNJ:TAJP156M006SNJ
- added D1: FIX, LED_SMD:LED_0805_2012Metric_Pad1.15x1.40mm_HandSolder, symbol Device:LED
- added D2: 1N5817, Diode_SMD:D_0805_2012Metric_Pad1.15x1.40mm_HandSolder, symbol Diode:1N5817
- added J1: CONUFL001-SMD-T, foot:LINX_CONUFL001-SMD-T, symbol Replica_NEO_6M_GPS-rescue:CONUFL001-SMD-T-CONUFL001-SMD-T
- added L1: 27uH, Inductor_SMD:L_0805_2012Metric_Pad1.15x1.40mm_HandSolder, symbol Device:L
- added R1, R3: 1K, Resistor_SMD:R_0805_2012Metric_Pad1.20x1.40mm_HandSolder, symbol Device:R
- added R2: 22R, Resistor_SMD:R_0805_2012Metric_Pad1.20x1.40mm_HandSolder, symbol Device:R
- added U1: TPS79133DBVR, foot:SOT95P280X145-5N, symbol Replica_NEO_6M_GPS-rescue:TPS79133DBVR-TPS79133DBVR
- added U2: NEO-6M-GPS, foot:XCVR_NEO-6M-GPS, symbol Replica_NEO_6M_GPS-rescue:NEO-6M-GPS-NEO-6M-GPS
- added U3: 24AA32A-I_MS, foot:SOP65P490X110-8N, symbol Replica_NEO_6M_GPS-rescue:24AA32A-I_MS-24AA32A-I_MS
Connections:
- net labels added: +3.3V, GND, RXD1, SCL2, SDA2, TXD1, VCC
- net labels removed: Earth
- wire segments 20 -> 87
- no-connect marks 0 -> 9
Other:
- note added: "Antenna"
- note added: "HEADER"
- note added: "Level shifting (5V <---> 3,3V)"
- note added: "NEO-6M-0-001\n752000358170\n1744\n0300 7"
- note added: "NOTA:"
- note added: "POWER MANAGEMENT"
- note added: "SERIAL EEPROM"
- note added: "T494B475K010"
- note added: "T494B475K010: Capacitor de tantalio, 4,7uF, 6,8V"
- note added: "UBLOX NEO 6M-V2"
- note added: "VCC range: 1,7V to 5,5V\nICC range: 0A to 3mA\n32-Byte Page Write Buffer"
- note added: "VCC range: 2,7V to 5,5V"
- note removed: "5V"
- note removed: "GND"
- note removed: "RXD1\n"
- note removed: "TXD1"
- moved on the sheet: H1, H2, H3, H4, H5, J2
